File: doc/pcb/synchro2/synchro2.kicad_pcb (KiCad board)
At the start: 2 copper layers, 40 x 40 mm, 37 parts, among them J1 Charging port, J2 Cell pad, M1 Motor_DC, Q1 BS170F, U1 TC1186, U2 STM32F030F4Px, U3 KTIR0711S, Y1 32.768

Commit message: hall sensor, updated scheme and pcb
Parts:
- removed U3: KTIR0711S, Package_DIP:DIP-4_W7.62mm
- added HALL: SS311PT, Package_TO_SOT_SMD:SOT-23, B.Cu at (219.2, 132.0)
- MOS: renamed from Q1; value BS170F -> IRLML0030TR
- R11: value 1k -> 15k
- R3: value 22R -> 470R
- STM32: renamed from U2; value STM32F030F4Px -> STM32F041F6Px
- moved R3 20.6 mm to (233.2, 108.2), turned to 0 degrees
- moved R11 0.91 mm to (233.2, 105.7), turned to 0 degrees
- renumbered J1 to CHARGING, Y1 to CRYSTAL, M1 to MOTOR, U1 to REG, J2 to Vcc
Connections:
- MOS pad 1: CLK -> Net-(Q1-Pad1)
- R11 pad 1: CLK -> Net-(Q1-Pad1)
- R3 pad 1: Net-(R3-Pad1) -> Net-(Q1-Pad1)
Routing:
- net Net-(R3-Pad1): track 12.4 -> 0.00 mm
- net CLK: track 35.9 -> 43.7 mm
- net Net-(Q1-Pad1): track 0.00 -> 7.23 mm
- net GND: track 19.4 -> 14.5 mm
- net DIO: track 28.4 -> 25.6 mm
Other:
- board text added: "v0.2"
- board text removed: "v0.1"
