File: doc/pcb/synchro2/synchro2.kicad_pcb (KiCad board)
At the start: 2 copper layers, 40 x 40 mm, 37 parts

Commit message: added connections for ADC
Parts:
- added C5: 100n, Capacitor_SMD:C_0603_1608Metric, B.Cu at (224.2, 103.3)
- added R12: 15k, Resistor_SMD:R_0603_1608Metric, B.Cu at (225.0, 105.9)
- added R13: 15k, Resistor_SMD:R_0603_1608Metric, B.Cu at (224.9, 107.5)
- ARM Cortex: renamed from STM32
- moved GND 4.05 mm to (234.4, 107.3)
- renumbered Vcc to J2, MOTOR to M1, MOS to Q1, REG to U1, HALL to U4
Connections:
- ARM Cortex pad 11: Net-(U2-Pad11) -> VBAT
Routing:
- net VBAT: track 0.00 -> 17.6 mm, vias 0 -> 1
- net +5V: track 54.3 -> 60.0 mm
- net GND: vias 2 -> 3
Other:
- board text added: "v0.3"
- board text removed: "v0.2"

Commit message: v0.4 pcb
Parts:
- moved C1 6.09 mm to (207.4, 127.2)
- moved U1 4.81 mm to (210.5, 128.0)
- moved R3 3.00 mm to (231.9, 105.5)
- moved R11 2.09 mm to (231.9, 104.0)
- renumbered J2 to BATT, U4 to HALL, M1 to MOTOR
Routing:
- net CLK: track 43.7 -> 47.2 mm
- net Net-(Q1-Pad1): track 7.23 -> 4.15 mm
- net +5V: track 60.0 -> 62.9 mm
- net Vcc: track 40.7 -> 38.9 mm
- net GND: track 14.5 -> 13.1 mm
Other:
- board size 40 x 40 mm -> 41.4 x 41.4 mm
- board text added: "v0.4"
- board text removed: "v0.3"
