File: doc/pcb/synchro2/synchro2.kicad_pcb (KiCad board)
At the start: 2 copper layers, 41.4 x 41.4 mm, 40 parts, among them Q1 IRLML0030TR, U1 TC1186

Commit message: new design
Parts:
- removed BATT: Cell pad, LED_SMD:LED_2512_6332Metric_Pad1.52x3.35mm_HandSolder
- removed CLK, DIO, GND, RST, Vcc: PinSocket_1x01_P2.54mm_Vertical, Connector_PinSocket_2.54mm:PinSocket_1x01_P2.54mm_Vertical
- removed MOTOR: Motor_DC, LED_SMD:LED_2816_7142Metric
- added BT1: Battery_Cell, Resistor_SMD:R_1206_3216Metric, B.Cu at (215.9, 125.3)
- added BT2: Battery_Cell, Resistor_SMD:R_1206_3216Metric, B.Cu at (216.0, 102.0)
- added J2: programming, Connector_PinHeader_1.27mm:PinHeader_1x05_P1.27mm_Vertical, F.Cu at (235.8, 104.6)
- added M1: Motor_DC, Resistor_SMD:R_1206_3216Metric, B.Cu at (219.1, 101.9)
- U1: value TC1186 -> TC1185-3.3VCT8
- moved Quartz1 0.20 mm to (223.7, 121.9)
- renumbered Cortex to Core1, CHARGING to J1, CRYSTAL to Quartz1, SET to SET1, HALL to U4, WAKE to WAKE1
Connections:
- Core1 pad 8: Net-(U2-Pad8) -> (no net)
- U1 pad 4: Net-(U1-Pad4) -> (no net)
Routing:
- net Vcc: track 38.9 -> 63.9 mm, vias 1 -> 3
- net DIO: track 25.6 -> 42.4 mm
- net GND: track 13.1 -> 22.7 mm, vias 3 -> 11
- net CLK: track 47.2 -> 56.7 mm, vias 2 -> 3
- net RST: track 19.0 -> 26.9 mm, vias 0 -> 2
- net +5V: track 62.9 -> 60.4 mm, vias 0 -> 1
- net Net-(Core1-Pad17): track 9.58 -> 10.9 mm
- net Net-(Core1-Pad18): track 7.61 -> 8.86 mm
- net Net-(Core1-Pad14): track 12.1 -> 13.1 mm
- net Net-(C4-Pad1): track 18.0 -> 18.7 mm
- net Net-(Core1-Pad12): track 16.0 -> 16.6 mm
- removed copper zone on F.Cu, net (none)
Other:
- board text added: "Designed by Bart"
- board text added: "SynChro Mk5"
- board text removed: "Bart's"
- board text removed: "SYNCHRO 2"
- board text removed: "v0.4"

Commit message: small pcb corrections
Parts:
- moved BT1 2.04 mm to (216.6, 127.2), turned to 180 degrees
- renumbered J1 to CHARGING, Core1 to Core, Quartz1 to Quartz, SET1 to SET, WAKE1 to WAKE
Routing:
- net GND: track 22.7 -> 18.6 mm
Changed lines of the file:
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@@
-(kicad_pcb (version 20171130) (host pcbnew "(5.1.4)-1")
+(kicad_pcb (version 20171130) (host pcbnew 5.1.4-1.fc30)
   (general
     (thickness 1.6)
     (drawings 32)
-    (tracks 290)
+    (tracks 287)
     (zones 0)
     (modules 37)
@@
   )
   (setup
-    (last_trace_width 0.4)
+    (last_trace_width 0.25)
     (user_trace_width 0.4)
     (trace_clearance 0.2)
@@
       (drillshape 0)
       (scaleselection 1)
-      (outputdirectory "output/v0.4/"))
+      (outputdirectory "output/v0.5"))
   )
   (net 0 "")
@@
     (descr "Crystal THT DS26 6.0mm length 2.0mm diameter http://www.microcrystal.com/images/_Product-Documentation/03_TF_metal_Packages/01_Datasheet/DS-Series.pdf")
     (tags ['DS26'])
-    (fp_text reference Quartz1 (at 3.15 3.85) (layer F.SilkS)
+    (fp_text reference Quartz (at 3.15 3.85) (layer F.SilkS)
       (effects (font (size 1 1) (thickness 0.15)))
     )
@@
     (tags "SPST button tactile switch")
     (attr smd)
-    (fp_text reference WAKE1 (at 0.05 3.1) (layer F.SilkS)
+    (fp_text reference WAKE (at 0.05 3.1) (layer F.SilkS)
       (effects (font (size 1 1) (thickness 0.15)))
     )
@@
     (descr "Through hole angled pin header, 1x02, 2.54mm pitch, 6mm pin length, single row")
     (tags "Through hole angled pin header THT 1x02 2.54mm single row")
-    (fp_text reference J1 (at 4.385 -2.27 45) (layer F.SilkS)
+    (fp_text reference CHARGING (at 4.385 -2.27 45) (layer F.SilkS)
       (effects (font (size 1 1) (thickness 0.15)))
     )
@@
     (tags "SSOP 0.65")
     (attr smd)
-    (fp_text reference Core1 (at 4.48 -0.6 180) (layer F.SilkS)
+    (fp_text reference Core (at 4.48 -0.6 180) (layer F.SilkS)
       (effects (font (size 0.8 0.8) (thickness 0.15)))
     )
@@
     (tags "SPST button tactile switch")
     (attr smd)
-    (fp_text reference SET1 (at -0.05 3.15) (layer F.SilkS)
+    (fp_text reference SET (at -0.05 3.15) (layer F.SilkS)
       (effects (font (size 1 1) (thickness 0.15)))
     )
@@
   )
   (module Resistor_SMD:R_1206_3216Metric (layer B.Cu)
-    (at 215.92 125.29 90)
+    (at 216.63 127.2 180)
     (descr "Resistor SMD 1206 (3216 Metric), square (rectangular) end terminal, IPC_7351 nominal, (Body size source: http://www.tortai-tech.com/upload/download/2011102023233369053.pdf), generated with kicad-footprint-generator")
     (tags resistor)
     (attr smd)
-    (fp_text reference BT1 (at 0 1.82 270) (layer B.SilkS)
-      (effects (font (size 1 1) (thickness 0.15)) (justify mirror))
-    )
-    (fp_text value Battery_Cell (at 0 -1.82 270) (layer B.Fab)
+    (fp_text reference BT1 (at 0 1.82 180) (layer B.SilkS)
+      (effects (font (size 1 1) (thickness 0.15)) (justify mirror))
+    )
+    (fp_text value Battery_Cell (at 0 -1.82 180) (layer B.Fab)
       (effects (font (size 1 1) (thickness 0.15)) (justify mirror))
     )
@@
     (fp_line (start 2.28 1.12) (end 2.28 -1.12) (layer B.CrtYd) (width 0.05))
     (fp_line (start 2.28 -1.12) (end -2.28 -1.12) (layer B.CrtYd) (width 0.05))
-    (fp_text user %R (at 0 0 270) (layer B.Fab)
+    (fp_text user %R (at 0 0 180) (layer B.Fab)
       (effects (font (size 0.8 0.8) (thickness 0.12)) (justify mirror))
     )
-    (pad 1 smd roundrect (at -1.4 0 90) (size 1.25 1.75) (layers B.Cu B.Paste B.Mask) (roundrect_rratio 0.2)
+    (pad 1 smd roundrect (at -1.4 0 180) (size 1.25 1.75) (layers B.Cu B.Paste B.Mask) (roundrect_rratio 0.2)
       (net 2 +5V))
-    (pad 2 smd roundrect (at 1.4 0 90) (size 1.25 1.75) (layers B.Cu B.Paste B.Mask) (roundrect_rratio 0.2)
+    (pad 2 smd roundrect (at 1.4 0 180) (size 1.25 1.75) (layers B.Cu B.Paste B.Mask) (roundrect_rratio 0.2)
       (net 1 GND))
     (model ${KISYS3DMOD}/Resistor_SMD.3dshapes/R_1206_3216Metric.wrl
@@
   (segment (start 207.3925 128.02) (end 207.38 128.0075) (width 0.4) (layer B.Cu) (net 1) (status 30))
   (segment (start 209.44 128.02) (end 207.3925 128.02) (width 0.4) (layer B.Cu) (net 1) (status 30))
-  (segment (start 213.74 128.02) (end 209.44 128.02) (width 0.4) (layer B.Cu) (net 1) (status 20))
-  (segment (start 213.94 127.82) (end 213.74 128.02) (width 0.4) (layer B.Cu) (net 1))
-  (segment (start 213.94 124.22) (end 213.94 127.82) (width 0.4) (layer B.Cu) (net 1))
-  (segment (start 215.92 123.89) (end 214.27 123.89) (width 0.4) (layer B.Cu) (net 1) (status 10))
-  (segment (start 214.27 123.89) (end 213.94 124.22) (width 0.4) (layer B.Cu) (net 1))
   (via (at 232.39 100.77) (size 1.5) (drill 0.8) (layers F.Cu B.Cu) (net 1))
   (via (at 230.89 99.79) (size 1.5) (drill 0.8) (layers F.Cu B.Cu) (net 1))
@@
   (segment (start 227.9 108.78) (end 228.42 109.3) (width 0.4) (layer F.Cu) (net 1))
   (segment (start 227.76 108.78) (end 227.9 108.78) (width 0.4) (layer F.Cu) (net 1))
+  (segment (start 214.41 128.02) (end 215.23 127.2) (width 0.4) (layer B.Cu) (net 1))
+  (segment (start 209.44 128.02) (end 214.41 128.02) (width 0.4) (layer B.Cu) (net 1))
   (via (at 211.95 106.16) (size 1.5) (drill 0.8) (layers F.Cu B.Cu) (net 2))
   (segment (start 216.682001 130.870001) (end 211.545001 130.870001) (width 0.4) (layer B.Cu) (net 2))
@@
   (segment (start 209.645 128.97) (end 209.44 128.97) (width 0.4) (layer B.Cu) (net 2) (status 30))
   (segment (start 211.545001 130.870001) (end 209.645 128.97) (width 0.4) (layer B.Cu) (net 2) (status 20))
-  (segment (start 217.280001 128.067501) (end 217.280001 130.272001) (width 0.4) (layer B.Cu) (net 2))
-  (segment (start 216.1125 126.9) (end 217.280001 128.067501) (width 0.4) (layer B.Cu) (net 2) (status 10))
   (segment (start 208.8025 126.4325) (end 209.44 127.07) (width 0.4) (layer B.Cu) (net 2) (status 20))
   (segment (start 207.38 126.4325) (end 208.8025 126.4325) (width 0.4) (layer B.Cu) (net 2) (status 10))
@@
   (segment (start 206.84605 109.746052) (end 208.363948 109.746052) (width 0.4) (layer B.Cu) (net 2))
   (segment (start 205.996051 110.596051) (end 206.84605 109.746052) (width 0.4) (layer B.Cu) (net 2) (status 10))
+  (segment (start 217.280001 127.949999) (end 218.03 127.2) (width 0.4) (layer B.Cu) (net 2))
+  (segment (start 217.280001 130.272001) (end 217.280001 127.949999) (width 0.4) (layer B.Cu) (net 2))
   (segment (start 230.775 120.35) (end 230.775 114.45) (width 0.4) (layer F.Cu) (net 3) (status 30))
   (segment (start 230.775 120.35) (end 230.775 122.675) (width 0.4) (layer F.Cu) (net 3) (status 10))
