File: doc/case/V3/base/base.kicad_pcb (KiCad board)
At the start: 2 copper layers, 43.9 x 52.1 mm, 0 parts

Commit message: new case
Other:
- board size 43.9 x 52.1 mm -> 51.9 x 52.1 mm
Changed lines of the file:
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@@
   (general
     (thickness 1.6)
-    (drawings 43)
+    (drawings 39)
     (tracks 0)
     (zones 0)
@@
     (uvia_drill 0.1)
   )
+  (gr_arc (start 216.53 73.47) (end 235.7065 56.01758) (angle 84.60916232) (layer Edge.Cuts) (width 0.05))
+  (gr_arc (start 216.53 73.47) (end 197.350001 90.919999) (angle 84.6) (layer Edge.Cuts) (width 0.05))
   (gr_line (start 231.336883 99.492832) (end 238.482403 98.357372) (layer Edge.Cuts) (width 0.05))
-  (gr_line (start 238.482403 98.357372) (end 235.718383 90.915252) (layer Edge.Cuts) (width 0.05))
+  (gr_line (start 238.482403 98.357372) (end 235.706843 90.922043) (layer Edge.Cuts) (width 0.05))
   (gr_line (start 201.735 99.5) (end 194.577597 98.357372) (layer Edge.Cuts) (width 0.05))
-  (gr_line (start 194.577597 98.357372) (end 197.352447 90.922688) (layer Edge.Cuts) (width 0.05))
+  (gr_line (start 194.577597 98.357372) (end 197.350001 90.919999) (layer Edge.Cuts) (width 0.05))
   (gr_line (start 231.325 47.44) (end 238.482403 48.582628) (layer Edge.Cuts) (width 0.05))
-  (gr_line (start 238.482403 48.582628) (end 235.707553 56.017312) (layer Edge.Cuts) (width 0.05))
+  (gr_line (start 238.482403 48.582628) (end 235.7065 56.01758) (layer Edge.Cuts) (width 0.05))
   (gr_line (start 201.723117 47.447168) (end 194.577597 48.582628) (layer Edge.Cuts) (width 0.05))
-  (gr_line (start 194.577597 48.582628) (end 197.341617 56.024748) (layer Edge.Cuts) (width 0.05))
-  (gr_line (start 235.7065 56.01758) (end 233.03 62.17) (layer Edge.Cuts) (width 0.05))
-  (gr_line (start 233.03 84.77) (end 235.718383 90.915252) (layer Edge.Cuts) (width 0.05))
-  (gr_line (start 200.03 84.77) (end 197.3535 90.92242) (layer Edge.Cuts) (width 0.05))
-  (gr_line (start 197.341617 56.024748) (end 200.03 62.17) (layer Edge.Cuts) (width 0.05))
+  (gr_line (start 194.577597 48.582628) (end 197.352447 56.017312) (layer Edge.Cuts) (width 0.05))
   (gr_circle (center 198.415883 96.673337) (end 199.685883 96.165337) (layer Edge.Cuts) (width 0.05))
   (gr_circle (center 234.656 96.666169) (end 233.386 96.158169) (layer Edge.Cuts) (width 0.05))
@@
   (gr_line (start 203.33 54.15) (end 203.33 64.15) (layer F.SilkS) (width 0.12))
   (gr_circle (center 216.53 73.47) (end 225.43 73.47) (layer F.SilkS) (width 0.12))
-  (gr_arc (start 238.82 73.47) (end 233.03 62.17) (angle -125.7397604) (layer Edge.Cuts) (width 0.05))
-  (gr_arc (start 194.24 73.47) (end 200.03 84.77) (angle -125.7397604) (layer Edge.Cuts) (width 0.05))
   (gr_line (start 204.03 51.97) (end 229.03 51.97) (layer Edge.Cuts) (width 0.05))
   (gr_line (start 229.03 51.97) (end 229.03 53.97) (layer Edge.Cuts) (width 0.05))

Commit message: new case
Other:
- board size 51.9 x 52.1 mm -> 51.9 x 52 mm
Changed lines of the file:
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@@
     (uvia_drill 0.1)
   )
-  (gr_arc (start 216.53 73.47) (end 235.7065 56.01758) (angle 84.60916232) (layer Edge.Cuts) (width 0.05))
-  (gr_arc (start 216.53 73.47) (end 197.350001 90.919999) (angle 84.6) (layer Edge.Cuts) (width 0.05))
-  (gr_line (start 231.336883 99.492832) (end 238.482403 98.357372) (layer Edge.Cuts) (width 0.05))
-  (gr_line (start 238.482403 98.357372) (end 235.706843 90.922043) (layer Edge.Cuts) (width 0.05))
-  (gr_line (start 201.735 99.5) (end 194.577597 98.357372) (layer Edge.Cuts) (width 0.05))
-  (gr_line (start 194.577597 98.357372) (end 197.350001 90.919999) (layer Edge.Cuts) (width 0.05))
-  (gr_line (start 231.325 47.44) (end 238.482403 48.582628) (layer Edge.Cuts) (width 0.05))
-  (gr_line (start 238.482403 48.582628) (end 235.7065 56.01758) (layer Edge.Cuts) (width 0.05))
-  (gr_line (start 201.723117 47.447168) (end 194.577597 48.582628) (layer Edge.Cuts) (width 0.05))
-  (gr_line (start 194.577597 48.582628) (end 197.352447 56.017312) (layer Edge.Cuts) (width 0.05))
-  (gr_circle (center 198.415883 96.673337) (end 199.685883 96.165337) (layer Edge.Cuts) (width 0.05))
-  (gr_circle (center 234.656 96.666169) (end 233.386 96.158169) (layer Edge.Cuts) (width 0.05))
-  (gr_circle (center 234.644117 50.266663) (end 233.374117 50.774663) (layer Edge.Cuts) (width 0.05))
+  (gr_arc (start 216.53 73.47) (end 236.122 56.48) (angle 81.86304929) (layer Edge.Cuts) (width 0.05))
+  (gr_arc (start 216.53 73.47) (end 196.932 90.46) (angle 81.87684461) (layer Edge.Cuts) (width 0.05))
+  (gr_line (start 203.978 47.45) (end 197.698 47.45) (layer Edge.Cuts) (width 0.05))
+  (gr_line (start 203.98 48.73) (end 203.978 47.45) (layer Edge.Cuts) (width 0.05))
+  (gr_line (start 197.698 99.49) (end 196.932 90.46) (layer Edge.Cuts) (width 0.05))
+  (gr_line (start 203.98 98.21) (end 203.978 99.49) (layer Edge.Cuts) (width 0.05))
+  (gr_line (start 229.082 98.21) (end 229.082 99.49) (layer Edge.Cuts) (width 0.05))
+  (gr_line (start 235.362 99.49) (end 236.122 90.46) (layer Edge.Cuts) (width 0.05))
+  (gr_line (start 197.698 47.45) (end 196.941244 56.469343) (layer Edge.Cuts) (width 0.05))
+  (gr_line (start 229.082 99.49) (end 235.362 99.49) (layer Edge.Cuts) (width 0.05))
+  (gr_line (start 235.362 47.45) (end 236.122 56.48) (layer Edge.Cuts) (width 0.05))
+  (gr_line (start 203.978 99.49) (end 197.698 99.49) (layer Edge.Cuts) (width 0.05))
+  (gr_line (start 229.083117 48.73) (end 229.082 47.45) (layer Edge.Cuts) (width 0.05))
+  (gr_line (start 229.082 47.45) (end 235.362 47.45) (layer Edge.Cuts) (width 0.05))
+  (gr_line (start 203.98 98.21) (end 229.082 98.21) (layer Edge.Cuts) (width 0.05))
+  (gr_circle (center 200.415883 96.673337) (end 201.783715 96.673337) (layer Edge.Cuts) (width 0.05))
+  (gr_circle (center 232.656 96.666169) (end 234.023832 96.666169) (layer Edge.Cuts) (width 0.05))
+  (gr_circle (center 232.644117 50.266663) (end 234.011949 50.266663) (layer Edge.Cuts) (width 0.05))
   (gr_circle (center 216.53 73.47) (end 216.22 73.31) (layer B.SilkS) (width 0.12))
-  (gr_line (start 230.41 96.97) (end 231.336883 99.492832) (layer Edge.Cuts) (width 0.05))
-  (gr_line (start 202.65 49.97) (end 201.723117 47.447168) (layer Edge.Cuts) (width 0.05))
-  (gr_line (start 230.39 49.97) (end 231.325 47.44) (layer Edge.Cuts) (width 0.05))
-  (gr_line (start 202.67 96.97) (end 201.735 99.5) (layer Edge.Cuts) (width 0.05))
-  (gr_circle (center 198.404 50.273831) (end 199.674 50.781831) (layer Edge.Cuts) (width 0.05))
+  (gr_circle (center 200.404 50.273831) (end 201.771832 50.273831) (layer Edge.Cuts) (width 0.05))
   (gr_line (start 229.73 82.79) (end 214.73 82.79) (layer F.SilkS) (width 0.12))
   (gr_line (start 229.73 92.79) (end 229.73 82.79) (layer F.SilkS) (width 0.12))
@@
   (gr_circle (center 216.53 73.47) (end 225.43 73.47) (layer F.SilkS) (width 0.12))
   (gr_line (start 204.03 51.97) (end 229.03 51.97) (layer Edge.Cuts) (width 0.05))
-  (gr_line (start 229.03 51.97) (end 229.03 53.97) (layer Edge.Cuts) (width 0.05))
-  (gr_line (start 204.03 53.97) (end 204.03 51.97) (layer Edge.Cuts) (width 0.05))
-  (gr_line (start 229.03 53.97) (end 204.03 53.97) (layer Edge.Cuts) (width 0.05))
+  (gr_line (start 229.03 49.97) (end 229.03 51.97) (layer Edge.Cuts) (width 0.05))
+  (gr_line (start 204.03 51.97) (end 204.03 49.97) (layer Edge.Cuts) (width 0.05))
+  (gr_line (start 229.03 49.97) (end 204.03 49.97) (layer Edge.Cuts) (width 0.05))
   (gr_line (start 229.03 94.97) (end 204.03 94.97) (layer Edge.Cuts) (width 0.05))
-  (gr_line (start 229.03 92.97) (end 229.03 94.97) (layer Edge.Cuts) (width 0.05))
-  (gr_line (start 204.03 92.97) (end 229.03 92.97) (layer Edge.Cuts) (width 0.05))
-  (gr_line (start 204.03 94.97) (end 204.03 92.97) (layer Edge.Cuts) (width 0.05))
-  (gr_line (start 230.39 49.97) (end 202.65 49.97) (layer Edge.Cuts) (width 0.05))
-  (gr_line (start 202.67 96.97) (end 230.41 96.97) (layer Edge.Cuts) (width 0.05))
+  (gr_line (start 229.03 94.97) (end 229.03 96.97) (layer Edge.Cuts) (width 0.05))
+  (gr_line (start 204.03 96.97) (end 229.03 96.97) (layer Edge.Cuts) (width 0.05))
+  (gr_line (start 204.03 96.97) (end 204.03 94.97) (layer Edge.Cuts) (width 0.05))
+  (gr_line (start 229.083117 48.73) (end 203.98 48.73) (layer Edge.Cuts) (width 0.05))
 )

Commit message: new case
Other:
- outline, holes or cut-outs redrawn
Changed lines of the file:
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@@
   (general
     (thickness 1.6)
-    (drawings 39)
+    (drawings 33)
     (tracks 0)
     (zones 0)
@@
     (uvia_drill 0.1)
   )
-  (gr_arc (start 216.53 73.47) (end 236.122 56.48) (angle 81.86304929) (layer Edge.Cuts) (width 0.05))
-  (gr_arc (start 216.53 73.47) (end 196.932 90.46) (angle 81.87684461) (layer Edge.Cuts) (width 0.05))
-  (gr_line (start 203.978 47.45) (end 197.698 47.45) (layer Edge.Cuts) (width 0.05))
-  (gr_line (start 203.98 48.73) (end 203.978 47.45) (layer Edge.Cuts) (width 0.05))
-  (gr_line (start 197.698 99.49) (end 196.932 90.46) (layer Edge.Cuts) (width 0.05))
-  (gr_line (start 203.98 98.21) (end 203.978 99.49) (layer Edge.Cuts) (width 0.05))
-  (gr_line (start 229.082 98.21) (end 229.082 99.49) (layer Edge.Cuts) (width 0.05))
-  (gr_line (start 235.362 99.49) (end 236.122 90.46) (layer Edge.Cuts) (width 0.05))
-  (gr_line (start 197.698 47.45) (end 196.941244 56.469343) (layer Edge.Cuts) (width 0.05))
-  (gr_line (start 229.082 99.49) (end 235.362 99.49) (layer Edge.Cuts) (width 0.05))
-  (gr_line (start 235.362 47.45) (end 236.122 56.48) (layer Edge.Cuts) (width 0.05))
-  (gr_line (start 203.978 99.49) (end 197.698 99.49) (layer Edge.Cuts) (width 0.05))
-  (gr_line (start 229.083117 48.73) (end 229.082 47.45) (layer Edge.Cuts) (width 0.05))
-  (gr_line (start 229.082 47.45) (end 235.362 47.45) (layer Edge.Cuts) (width 0.05))
-  (gr_line (start 203.98 98.21) (end 229.082 98.21) (layer Edge.Cuts) (width 0.05))
+  (gr_line (start 234.168 99.49) (end 237.308 88.99) (layer Edge.Cuts) (width 0.05))
+  (gr_line (start 234.168 47.45) (end 237.308 57.95) (layer Edge.Cuts) (width 0.05))
+  (gr_line (start 229.082 47.45) (end 234.168 47.45) (layer Edge.Cuts) (width 0.05))
+  (gr_line (start 198.892 99.49) (end 195.752 88.99) (layer Edge.Cuts) (width 0.05))
+  (gr_line (start 229.082 99.49) (end 198.892 99.49) (layer Edge.Cuts) (width 0.05))
+  (gr_line (start 229.082 47.45) (end 198.892 47.45) (layer Edge.Cuts) (width 0.05))
+  (gr_line (start 198.892 47.45) (end 195.751999 57.950002) (layer Edge.Cuts) (width 0.05))
+  (gr_line (start 229.082 99.49) (end 234.168 99.49) (layer Edge.Cuts) (width 0.05))
+  (gr_arc (start 216.53 73.47) (end 237.308 57.95) (angle 73.51533497) (layer Edge.Cuts) (width 0.05))
+  (gr_arc (start 216.53 73.47) (end 195.752 88.99) (angle 73.51533011) (layer Edge.Cuts) (width 0.05))
   (gr_circle (center 200.415883 96.673337) (end 201.783715 96.673337) (layer Edge.Cuts) (width 0.05))
   (gr_circle (center 232.656 96.666169) (end 234.023832 96.666169) (layer Edge.Cuts) (width 0.05))
@@
   (gr_line (start 204.03 96.97) (end 229.03 96.97) (layer Edge.Cuts) (width 0.05))
   (gr_line (start 204.03 96.97) (end 204.03 94.97) (layer Edge.Cuts) (width 0.05))
-  (gr_line (start 229.083117 48.73) (end 203.98 48.73) (layer Edge.Cuts) (width 0.05))
 )
