File: doc/case/V3/base/base.kicad_pcb (KiCad board)
At the start: 2 copper layers, 51.9 x 52 mm, 0 parts

Commit message: new case
Other:
- board text added: "Designed by Bart"
- board text added: "SynChro Mk5"
Changed lines of the file:
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@@
-(kicad_pcb (version 20171130) (host pcbnew 5.1.4-1.fc30)
+(kicad_pcb (version 20171130) (host pcbnew "(5.1.4)-1")
   (general
     (thickness 1.6)
-    (drawings 33)
+    (drawings 35)
     (tracks 0)
     (zones 0)
@@
     (solder_mask_min_width 0.25)
     (aux_axis_origin 0 0)
-    (visible_elements FFFFFF7F)
+    (visible_elements 7FFFFFFF)
     (pcbplotparams
       (layerselection 0x01000_7ffffffe)
@@
     (uvia_drill 0.1)
   )
+  (gr_text "Designed\n  by Bart" (at 223.08 76.63) (layer B.SilkS)
+    (effects (font (size 1 1) (thickness 0.15)) (justify mirror))
+  )
+  (gr_text "SynChro Mk5" (at 217.11 71.03) (layer B.SilkS)
+    (effects (font (size 2 2) (thickness 0.3)) (justify mirror))
+  )
   (gr_line (start 234.168 99.49) (end 237.308 88.99) (layer Edge.Cuts) (width 0.05))
   (gr_line (start 234.168 47.45) (end 237.308 57.95) (layer Edge.Cuts) (width 0.05))
@@
   (gr_circle (center 232.656 96.666169) (end 234.023832 96.666169) (layer Edge.Cuts) (width 0.05))
   (gr_circle (center 232.644117 50.266663) (end 234.011949 50.266663) (layer Edge.Cuts) (width 0.05))
-  (gr_circle (center 216.53 73.47) (end 216.22 73.31) (layer B.SilkS) (width 0.12))
+  (gr_circle (center 216.53 73.47) (end 216.878855 73.47) (layer Cmts.User) (width 0.12))
   (gr_circle (center 200.404 50.273831) (end 201.771832 50.273831) (layer Edge.Cuts) (width 0.05))
   (gr_line (start 229.73 82.79) (end 214.73 82.79) (layer F.SilkS) (width 0.12))
