File: doc/pcb/ChronoMatic/ChronoMatic.sch (KiCad schematic (older format))
At the start: 27 parts, among them J1 Conn_01x05, Q1 Q_Photo_NPN, SW1 SET, SW2 CLEAR, U1 STM32F030F4Px, Y1 7.3728

Commit message: new design
Parts:
- removed D8: LED, LED_SMD:LED_1806_4516Metric_Castellated, symbol Device:LED
- removed J1: Conn_01x05, Connector_PinHeader_2.54mm:PinHeader_1x05_P2.54mm_Vertical, symbol Connector_Generic:Conn_01x05
- removed Q1: Q_Photo_NPN, LED_SMD:LED_1806_4516Metric_Castellated, symbol Device:Q_Photo_NPN
- added BT2: Battery_Cell, Resistor_SMD:R_1206_3216Metric, symbol Device:Battery_Cell
- added C1, C2: 100n, Capacitor_SMD:C_0603_1608Metric, symbol Device:C
- added C5: 2.2u, Capacitor_SMD:C_0603_1608Metric, symbol Device:C
- added J1: Charging port, Connector_PinHeader_2.54mm:PinHeader_1x02_P2.54mm_Vertical, symbol Connector:Conn_01x02_Female
- added J2: Conn_01x05_Female, Connector_PinHeader_1.27mm:PinHeader_1x05_P1.27mm_Vertical, symbol Connector:Conn_01x05_Female
- added M1: Motor_DC, Resistor_SMD:R_1206_3216Metric, symbol Motor:Motor_DC
- added Q1: IRLML0030TR, Package_TO_SOT_SMD:SOT-23, symbol Transistor_FET:BS170F
- added R11: 15k, Resistor_SMD:R_0603_1608Metric, symbol Device:R
- added R12, R13: 100k, Resistor_SMD:R_0603_1608Metric, symbol Device:R
- added U1: TC1185-3.3VCT8, Package_TO_SOT_SMD:SOT-23-5, symbol Regulator_Linear:TC1186
- added U4: SS311PT, Package_TO_SOT_SMD:SOT-23, symbol Sensor_Magnetic:A1104LLHL
- BT1: footprint Battery:BatteryHolder_Keystone_1060_1x2032 -> Resistor_SMD:R_1206_3216Metric
- C3: renamed from C1; value 22p -> 10p
- C4: renamed from C2; value 22p -> 10p
- R10, R4, R5, R6, R7, R8, R9: value 220R -> 1k
- R3: value 22R -> 220R
- SW1: value SET -> WAKE; footprint Button_Switch_SMD:SW_SPST_B3S-1000 -> Button_Switch_SMD:SW_SPST_CK_RS282G05A3
- SW2: value CLEAR -> SET; footprint Button_Switch_SMD:SW_SPST_B3S-1000 -> Button_Switch_SMD:SW_SPST_CK_RS282G05A3
- U2: renamed from U1; value STM32F030F4Px -> STM32F041F6Px
- Y1: value 7.3728 -> 32.768; footprint Crystal:Crystal_HC49-U_Vertical -> Crystal:Crystal_DS26_D2.0mm_L6.0mm_Horizontal
Connections:
- net labels added: +5V, MOTOR, VBAT
- net labels removed: +3V3, clk, dio, gnd
- wire segments 75 -> 104
Other:
- moved on the sheet: BT1
