File: doc/case/V3/ring/ring.kicad_pcb (KiCad board)
At the start: 2 copper layers, 51.9 x 52.1 mm, 0 parts

Commit message: new case
Other:
- outline, holes or cut-outs redrawn
Changed lines of the file:
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@@
   (gr_arc (start 169.418 102.87) (end 188.5945 85.41758) (angle 84.60916232) (layer Edge.Cuts) (width 0.05))
   (gr_line (start 182.817999 125.069999) (end 184.224883 128.892832) (layer Edge.Cuts) (width 0.05))
-  (gr_circle (center 169.418 102.87) (end 169.418 82.554622) (layer Edge.Cuts) (width 0.05))
+  (gr_circle (center 169.418 102.87) (end 187.418 102.87) (layer Edge.Cuts) (width 0.05))
   (gr_line (start 156.029884 125.077167) (end 154.623 128.9) (layer Edge.Cuts) (width 0.05))
   (gr_arc (start 169.418 102.87) (end 182.817999 125.069999) (angle 62.2) (layer Edge.Cuts) (width 0.05))

Commit message: new case
Other:
- board size 51.9 x 52.1 mm -> 51.9 x 52 mm
Changed lines of the file:
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@@
       (padsonsilk false)
       (subtractmaskfromsilk false)
-      (outputformat 1)
+      (outputformat 3)
       (mirror false)
       (drillshape 0)
@@
     (uvia_drill 0.1)
   )
-  (gr_line (start 147.465597 77.982628) (end 150.240447 85.417312) (layer Edge.Cuts) (width 0.05))
-  (gr_line (start 154.611117 76.847168) (end 147.465597 77.982628) (layer Edge.Cuts) (width 0.05))
-  (gr_line (start 147.47748 127.76454) (end 150.238001 120.319999) (layer Edge.Cuts) (width 0.05))
-  (gr_line (start 154.623 128.9) (end 147.47748 127.76454) (layer Edge.Cuts) (width 0.05))
-  (gr_line (start 191.370403 127.757372) (end 188.594843 120.322043) (layer Edge.Cuts) (width 0.05))
-  (gr_line (start 184.224883 128.892832) (end 191.370403 127.757372) (layer Edge.Cuts) (width 0.05))
-  (gr_line (start 184.213 76.84) (end 191.35852 77.97546) (layer Edge.Cuts) (width 0.05))
-  (gr_line (start 182.806116 80.662833) (end 184.213 76.84) (layer Edge.Cuts) (width 0.05))
+  (gr_line (start 156.87 80.17) (end 156.866 76.85) (layer Edge.Cuts) (width 0.05))
+  (gr_line (start 156.866 76.85) (end 150.586 76.85) (layer Edge.Cuts) (width 0.05))
+  (gr_line (start 150.586 76.85) (end 149.829244 85.869343) (layer Edge.Cuts) (width 0.05))
+  (gr_line (start 156.861407 125.557458) (end 156.866 128.89) (layer Edge.Cuts) (width 0.05))
+  (gr_line (start 156.866 128.89) (end 150.586 128.89) (layer Edge.Cuts) (width 0.05))
+  (gr_line (start 150.586 128.89) (end 149.82 119.86) (layer Edge.Cuts) (width 0.05))
+  (gr_line (start 181.97 125.56) (end 181.97 128.89) (layer Edge.Cuts) (width 0.05))
+  (gr_line (start 181.97 128.89) (end 188.25 128.89) (layer Edge.Cuts) (width 0.05))
+  (gr_line (start 188.25 128.89) (end 189.01 119.86) (layer Edge.Cuts) (width 0.05))
+  (gr_line (start 188.25 76.85) (end 189.01 85.88) (layer Edge.Cuts) (width 0.05))
+  (gr_line (start 181.97 76.85) (end 188.25 76.85) (layer Edge.Cuts) (width 0.05))
+  (gr_line (start 181.969063 80.171694) (end 181.97 76.85) (layer Edge.Cuts) (width 0.05))
   (gr_text . (at 152.6391 112.2632 120) (layer F.SilkS)
     (effects (font (size 4 4) (thickness 0.25)))
@@
     (effects (font (size 4 4) (thickness 0.25)))
   )
-  (gr_circle (center 151.303883 126.073337) (end 152.573883 125.565337) (layer Edge.Cuts) (width 0.05))
-  (gr_circle (center 187.544 126.066169) (end 186.274 125.558169) (layer Edge.Cuts) (width 0.05))
-  (gr_circle (center 187.532117 79.666663) (end 186.262117 80.174663) (layer Edge.Cuts) (width 0.05))
-  (gr_circle (center 151.292 79.673831) (end 152.562 80.181831) (layer Edge.Cuts) (width 0.05))
-  (gr_arc (start 169.418 102.87) (end 150.238001 120.319999) (angle 84.6) (layer Edge.Cuts) (width 0.05))
-  (gr_line (start 156.018001 80.670001) (end 154.611117 76.847168) (layer Edge.Cuts) (width 0.05))
-  (gr_arc (start 169.418 102.87) (end 188.5945 85.41758) (angle 84.60916232) (layer Edge.Cuts) (width 0.05))
-  (gr_line (start 182.817999 125.069999) (end 184.224883 128.892832) (layer Edge.Cuts) (width 0.05))
+  (gr_circle (center 153.303883 126.073337) (end 154.671715 126.073337) (layer Edge.Cuts) (width 0.05))
+  (gr_circle (center 185.544 126.066169) (end 186.911832 126.066169) (layer Edge.Cuts) (width 0.05))
+  (gr_circle (center 185.532117 79.666663) (end 186.899949 79.666663) (layer Edge.Cuts) (width 0.05))
+  (gr_circle (center 153.292 79.673831) (end 154.659832 79.673831) (layer Edge.Cuts) (width 0.05))
+  (gr_arc (start 169.418 102.87) (end 149.82 119.86) (angle 81.87684461) (layer Edge.Cuts) (width 0.05))
+  (gr_arc (start 169.418 102.87) (end 189.01 85.88) (angle 81.86304929) (layer Edge.Cuts) (width 0.05))
   (gr_circle (center 169.418 102.87) (end 187.418 102.87) (layer Edge.Cuts) (width 0.05))
-  (gr_line (start 156.029884 125.077167) (end 154.623 128.9) (layer Edge.Cuts) (width 0.05))
-  (gr_arc (start 169.418 102.87) (end 182.817999 125.069999) (angle 62.2) (layer Edge.Cuts) (width 0.05))
-  (gr_arc (start 169.418 102.87) (end 156.018001 80.670001) (angle 62.2) (layer Edge.Cuts) (width 0.05))
-  (gr_line (start 191.35852 77.97546) (end 188.5945 85.41758) (layer Edge.Cuts) (width 0.05))
+  (gr_arc (start 169.418 102.87) (end 181.97 125.56) (angle 57.91391902) (layer Edge.Cuts) (width 0.05))
+  (gr_arc (start 169.418 102.87) (end 156.87 80.17) (angle 57.87320241) (layer Edge.Cuts) (width 0.05))
   (gr_circle (center 169.418 102.87) (end 169.108 102.71) (layer B.SilkS) (width 0.12))
 )

Commit message: new case
Other:
- outline, holes or cut-outs redrawn
Changed lines of the file:
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@@
   (general
     (thickness 1.6)
-    (drawings 46)
+    (drawings 53)
     (tracks 0)
     (zones 0)
@@
       (drillshape 0)
       (scaleselection 1)
-      (outputdirectory "output/dxf/"))
+      (outputdirectory "/home/bartosz/projekty/arm/workspace/Spinner/doc/case/V3/ring/output/"))
   )
   (net 0 "")
@@
     (uvia_drill 0.1)
   )
+  (gr_line (start 156.866 128.89) (end 151.78 128.89) (layer Edge.Cuts) (width 0.05))
+  (gr_line (start 151.78 128.89) (end 148.64 118.39) (layer Edge.Cuts) (width 0.05))
+  (gr_line (start 181.97 128.89) (end 187.056 128.89) (layer Edge.Cuts) (width 0.05))
+  (gr_line (start 187.056 128.89) (end 190.196 118.39) (layer Edge.Cuts) (width 0.05))
+  (gr_line (start 181.97 76.85) (end 187.056 76.85) (layer Edge.Cuts) (width 0.05))
+  (gr_line (start 187.056 76.85) (end 190.196 87.35) (layer Edge.Cuts) (width 0.05))
+  (gr_line (start 156.78 175.72) (end 156.78 125.54) (layer Cmts.User) (width 0.15))
+  (gr_line (start 181.91 175.72) (end 181.91 125.61) (layer Cmts.User) (width 0.15))
+  (gr_line (start 156.78 14.77) (end 156.97 14.77) (layer Cmts.User) (width 0.15))
+  (gr_line (start 156.78 80.14) (end 156.78 14.77) (layer Cmts.User) (width 0.15))
+  (gr_line (start 181.91 175.72) (end 156.78 175.72) (layer Cmts.User) (width 0.15))
+  (gr_line (start 181.91 14.77) (end 181.91 80.07) (layer Cmts.User) (width 0.15))
+  (gr_line (start 156.97 14.77) (end 181.91 14.77) (layer Cmts.User) (width 0.15))
   (gr_line (start 156.87 80.17) (end 156.866 76.85) (layer Edge.Cuts) (width 0.05))
-  (gr_line (start 156.866 76.85) (end 150.586 76.85) (layer Edge.Cuts) (width 0.05))
-  (gr_line (start 150.586 76.85) (end 149.829244 85.869343) (layer Edge.Cuts) (width 0.05))
+  (gr_line (start 156.866 76.85) (end 151.78 76.85) (layer Edge.Cuts) (width 0.05))
+  (gr_line (start 151.78 76.85) (end 148.639999 87.350002) (layer Edge.Cuts) (width 0.05))
   (gr_line (start 156.861407 125.557458) (end 156.866 128.89) (layer Edge.Cuts) (width 0.05))
-  (gr_line (start 156.866 128.89) (end 150.586 128.89) (layer Edge.Cuts) (width 0.05))
-  (gr_line (start 150.586 128.89) (end 149.82 119.86) (layer Edge.Cuts) (width 0.05))
   (gr_line (start 181.97 125.56) (end 181.97 128.89) (layer Edge.Cuts) (width 0.05))
-  (gr_line (start 181.97 128.89) (end 188.25 128.89) (layer Edge.Cuts) (width 0.05))
-  (gr_line (start 188.25 128.89) (end 189.01 119.86) (layer Edge.Cuts) (width 0.05))
-  (gr_line (start 188.25 76.85) (end 189.01 85.88) (layer Edge.Cuts) (width 0.05))
-  (gr_line (start 181.97 76.85) (end 188.25 76.85) (layer Edge.Cuts) (width 0.05))
   (gr_line (start 181.969063 80.171694) (end 181.97 76.85) (layer Edge.Cuts) (width 0.05))
   (gr_text . (at 152.6391 112.2632 120) (layer F.SilkS)
@@
   (gr_circle (center 185.532117 79.666663) (end 186.899949 79.666663) (layer Edge.Cuts) (width 0.05))
   (gr_circle (center 153.292 79.673831) (end 154.659832 79.673831) (layer Edge.Cuts) (width 0.05))
-  (gr_arc (start 169.418 102.87) (end 149.82 119.86) (angle 81.87684461) (layer Edge.Cuts) (width 0.05))
-  (gr_arc (start 169.418 102.87) (end 189.01 85.88) (angle 81.86304929) (layer Edge.Cuts) (width 0.05))
+  (gr_arc (start 169.418 102.87) (end 148.64 118.39) (angle 73.51533011) (layer Edge.Cuts) (width 0.05))
+  (gr_arc (start 169.418 102.87) (end 190.196 87.35) (angle 73.51533497) (layer Edge.Cuts) (width 0.05))
   (gr_circle (center 169.418 102.87) (end 187.418 102.87) (layer Edge.Cuts) (width 0.05))
   (gr_arc (start 169.418 102.87) (end 181.97 125.56) (angle 57.91391902) (layer Edge.Cuts) (width 0.05))

Commit message: new case
Other:
- board text added: "Designed by Bart"
- board text added: "Mk5"
- board text added: "SynChro"
- board text removed: "12"

Commit message: new design
Other:
- board text removed: "Designed by Bart"
Changed lines of the file:
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@@
-(kicad_pcb (version 20171130) (host pcbnew "(5.1.4)-1")
+(kicad_pcb (version 20171130) (host pcbnew 5.1.4-1.fc30)
   (general
     (thickness 1.6)
-    (drawings 172)
+    (drawings 171)
     (tracks 0)
     (zones 0)
@@
     (uvia_drill 0.1)
   )
-  (gr_text "Designed\n  by Bart" (at 171.91736 83.9089) (layer F.SilkS)
-    (effects (font (size 0.5 0.5) (thickness 0.1)))
-  )
-  (gr_text Mk5 (at 166.39794 84.0486) (layer F.SilkS)
+  (gr_text Mk5 (at 169.418 122.174) (layer F.SilkS)
     (effects (font (size 1 1) (thickness 0.15)))
   )
   (gr_circle (center 169.418 102.87) (end 194.357647 102.87) (layer F.SilkS) (width 0.15))
-  (gr_text SynChro (at 169.4053 81.37652) (layer F.SilkS)
+  (gr_text SynChro (at 169.418 81.026) (layer F.SilkS)
     (effects (font (size 1.5 1.5) (thickness 0.3)))
   )
